Commit message: Added camera

File: cr5_ws/src/CR5_ROS/dobot_description/urdf/cr5_robot_gazebo-new-old.urdf (robot description, URDF)
Before this commit: robot cr5_robot, 11 links, 10 joints
Links:
- link wrist_rgbd_camera_link: mass 0.001 -> 0.05; geometry collision box size=0.04 0.04 0.03; visual box size=0.04 0.04 0.03
Joints:
- joint wrist_rgbd_camera_joint: origin xyz=0 -0.055 0 rpy=1.5708 -1.5708 0 -> xyz=0 0.14 0.08 rpy=0 1.5708 0
