Commit message: fix: fixed camera positioning

File: cr5_ws/src/CR5_ROS/dobot_description/urdf/cr5_robot_gazebo.urdf (robot description, URDF)
Before this commit: robot cr5_robot, 11 links, 10 joints
Joints:
- joint wrist_rgbd_camera_joint: origin xyz=0 0.14 0.08 rpy=0 1.5708 0 -> xyz=0 0.12 0.08 rpy=0 1.5708 0

Commit message: fix: repair Gazebo wrist camera simulation

File: cr5_ws/src/CR5_ROS/dobot_description/urdf/cr5_robot_gazebo.urdf (robot description, URDF)
Before this commit: robot cr5_robot, 11 links, 10 joints
Joints:
- joint wrist_rgbd_camera_optical_joint: origin xyz=0 0 0 rpy=-1.5708 0 -1.5708 -> xyz=0.04 0 0 rpy=-1.5708 0 -1.5708
